File: phase-detector.kicad_pcb (KiCad board)
At the start: 4 copper layers, 90.8 x 86.3 mm, 268 parts, among them J1 Conn_Coaxial_Small, J2 Conn_Coaxial_Small, J3 Conn_Coaxial_Small, J4 Conn_Coaxial_Small, J5 Conn_Coaxial_Small, J6 Conn_Coaxial_Small, J7 Conn_01x14_Socket, Q1 BFP740F, Q2 BFP740F, Q3 BFP740F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

Commit message: Rev 1 ready for review
Parts:
- removed U1: ICM-20948, Sensor_Motion:InvenSense_QFN-24_3x3mm_P0.4mm
- added C1: 100nF, Capacitor_SMD:C_0402_1005Metric, F.Cu at (98.0, 105.0)
- added C2: 10uF, Capacitor_SMD:C_0805_2012Metric, F.Cu at (96.1, 103.0)
- added TP1: INT_2, phase-detector:Test_Via, F.Cu at (97.1, 106.7)
- added TP10: ~{IRQ}, phase-detector:Test_Via, F.Cu at (82.3, 79.6)
- added TP11: ~{IRQ}, phase-detector:Test_Via, F.Cu at (108.6, 54.0)
- added TP12: ~{IRQ}, phase-detector:Test_Via, F.Cu at (140.4, 71.5)
- added TP13: ~{IRQ}, phase-detector:Test_Via, F.Cu at (135.6, 109.7)
- added TP2: DRDY, phase-detector:Test_Via, F.Cu at (98.5, 102.3)
- added TP3: INT_1, phase-detector:Test_Via, F.Cu at (104.1, 106.8)
- added TP4: Vref, phase-detector:Test_Via, F.Cu at (108.7, 107.4)
- added TP5: Vref, phase-detector:Test_Via, F.Cu at (91.4, 88.8)
- added TP6: Vref, phase-detector:Test_Via, F.Cu at (103.5, 65.7)
- added TP7: Vref, phase-detector:Test_Via, F.Cu at (128.7, 70.8)
- added TP8: Vref, phase-detector:Test_Via, F.Cu at (133.0, 95.9)
- added TP9: ~{IRQ}, phase-detector:Test_Via, F.Cu at (96.8, 114.6)
- added U14: LSM303C, Package_LGA:LGA-12_2x2mm_P0.5mm, F.Cu at (100.0, 104.0)
- C10, C117, C121, C130, C134, C52, C75: value 220 nF -> 220nF
- C105, C109, C110, C114, C12, C123, C127, C16, C45, C49, C68, C72: value C -> 1.2pF
- C106, C108, C111, C113, C124, C126, C13, C15, C46, C48, C69, C71: value C -> 1nF
- C107, C112, C125, C14, C47, C70: value C -> 0.36pF
- C11, C118, C122, C131, C135, C53, C76: value 3.3 pF -> 4.3 pF
- C115, C119, C128, C132, C50, C73, C8: value 220 nF -> 140nF
- C116, C120, C129, C133, C51, C74, C9: value 43 pF -> 10pF
- C136, C137, C138, C139: value 10nF -> 100pF
- C17, C18, C19, C20, C31, C32, C33, C34, C54, C55, C56, C57, C77, C78, C79, C80, C86, C87, C88, C89: value C_Small -> 1nF
- C24, C25, C38, C39, C61, C62, C84, C85, C93, C94: value C_Small -> ~
- C5: value 100nF -> 220nF
- L1, L16, L25, L40, L43, L51, L54: value 200 nF -> 130nH
- L11, L15, L20, L24, L30, L34, L35, L39, L4, L46, L50, L8: value L -> 1uH
- L12, L14, L21, L23, L31, L33, L36, L38, L47, L49, L5, L7: value L -> 1.2nH
- L13, L22, L32, L37, L48, L6: value L -> 3.3uH
- L17, L2, L26, L41, L44, L52, L55: value 200 nF -> 260nH
- L18, L27, L3, L42, L45, L53, L56: value 200 nF -> 30nH
- R16, R22, R31, R34, R37, R40, R7: value 20k -> 100k
- R17, R23, R32, R35, R38, R41, R8: value 10 -> 50
- R18, R24, R33, R36, R39, R42, R9: value 50 -> ~
- R43, R44, R45, R46: value 50 -> 75
- moved C139 37.5 mm to (90.0, 82.8), turned to 180 degrees
- moved C138 36.7 mm to (90.0, 81.8), turned to 180 degrees
- moved R46 36.7 mm to (92.0, 82.8)
- moved C137 36.1 mm to (90.0, 80.8), turned to 180 degrees
- moved R45 36.0 mm to (92.0, 81.8)
- moved C136 35.4 mm to (90.0, 79.8), turned to 180 degrees
- moved R44 35.3 mm to (92.0, 80.8)
- moved R43 34.5 mm to (92.0, 79.8)
- moved X1 4.94 mm to (100.0, 99.5)
- moved C5 3.60 mm to (100.0, 102.2), turned to 180 degrees
- moved C93 2.24 mm to (132.2, 98.6), turned to 72 degrees
- moved C84 2.24 mm to (131.0, 71.7), turned to 144 degrees
- moved C61 2.24 mm to (105.3, 64.3), turned to -144 degrees
- moved C24 2.24 mm to (106.5, 108.0), turned to 0 degrees
- moved C38 2.24 mm to (90.2, 86.8), turned to -72 degrees
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Connections:
- C5 pad 1: GND -> Net-(U14-C1)
- C5 pad 2: Net-(U1-REGOUT) -> GND
- J7 pad 10: CS3 -> CS4
- J7 pad 11: CS4 -> CS1
- J7 pad 12: CS5 -> CS2
- J7 pad 2: MISO -> SCK
- J7 pad 3: MOSI -> MISO
- J7 pad 4: MCLK_EN -> MOSI
- J7 pad 5: SCK -> MCLK_EN
- J7 pad 6: GND -> CS6
- J7 pad 7: CS0 -> CS5
- J7 pad 8: CS1 -> CS0
- J7 pad 9: CS2 -> CS3
- U12 pad 14: Net-(U12-SDO) -> MISO
- U12 pad 3: /ADC3/CH0 -> /AD8305/V_MAG
- U13 pad 14: Net-(U13-SDO) -> MISO
- U13 pad 3: /ADC4/CH0 -> /AD8306/V_MAG
- U5 pad 14: Net-(U5-SDO) -> MISO
- U5 pad 3: /ADC/CH0 -> /AD8302/V_MAG
- U7 pad 14: Net-(U7-SDO) -> MISO
- U7 pad 3: /ADC1/CH0 -> /AD8303/V_MAG
- U9 pad 14: Net-(U9-SDO) -> MISO
- U9 pad 3: /ADC2/CH0 -> /AD8304/V_MAG
Routing:
- net +3.3V-A: track 84.7 -> 282.7 mm, vias 16 -> 23
- net +3.3V-D: track 19.5 -> 211.8 mm, vias 3 -> 9
- net MCLK: track 0.00 -> 182.2 mm, vias 0 -> 7
- net MISO: track 13.6 -> 179.7 mm, vias 1 -> 6
- net MOSI: track 10.8 -> 175.9 mm, vias 1 -> 7
- net SCK: track 12.8 -> 166.1 mm, vias 1 -> 7
- net CS3: track 0.00 -> 55.1 mm, vias 0 -> 1
- net CS2: track 0.00 -> 35.9 mm, vias 0 -> 1
- net CS4: track 0.00 -> 35.5 mm, vias 0 -> 2
- net CS1: track 0.00 -> 22.3 mm, vias 0 -> 1
- net CS0: track 0.00 -> 18.8 mm, vias 0 -> 1
- net CS6: track 0.00 -> 10.2 mm, vias 0 -> 1
- net GND: track 0.90 -> 8.24 mm, vias 837 -> 786
- net /AD8305/V_REF: track 0.00 -> 5.77 mm
- net /AD8302/V_REF: track 0.00 -> 5.65 mm
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- added copper zone on In2.Cu, net GND
Other:
- board text added: "0"
- board text added: "1"
- board text added: "2"
- board text added: "2024-11-30"
- board text added: "3"
- board text added: "4"
- board text added: "Gavin Ford"
- board text added: "Rev 1"
- board text added: "WPI HPRC"
- board text added: "x"
- board text added: "y"

Commit message: added logo
Parts:
- added kibuzzard-674BE006: G***, kibuzzard-674BE006, F.Cu at (113.1, 77.1)
