File: AD8302.kicad_sch (KiCad schematic)
At the start: 13 parts, among them U6 AD8302

Commit message: Rev 1 ready for review
Parts:
- C31, C32, C33, C34: value C_Small -> 1nF
- C38, C39: value C_Small -> ~; now not fitted; now left out of the parts list
Changed lines of the file:
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@@
 			)
 		)
-		(property "Value" "C_Small"
+		(property "Value" "1nF"
 			(at 125.7363 107.95 90)
 			(effects
@@
 			)
 		)
-		(property "Value" "C_Small"
+		(property "Value" "1nF"
 			(at 125.7363 100.33 90)
 			(effects
@@
 		(unit 1)
 		(exclude_from_sim no)
-		(in_bom yes)
-		(on_board yes)
-		(dnp no)
+		(in_bom no)
+		(on_board yes)
+		(dnp yes)
 		(property "Reference" "C38"
 			(at 162.56 87.884 90)
@@
 			)
 		)
-		(property "Value" "C_Small"
+		(property "Value" "~"
 			(at 161.29 85.344 90)
 			(effects
@@
 		(unit 1)
 		(exclude_from_sim no)
-		(in_bom yes)
-		(on_board yes)
-		(dnp no)
+		(in_bom no)
+		(on_board yes)
+		(dnp yes)
 		(property "Reference" "C39"
 			(at 162.56 99.314 90)
@@
 			)
 		)
-		(property "Value" "C_Small"
+		(property "Value" "~"
 			(at 161.29 96.774 90)
 			(effects
@@
 			)
 		)
-		(property "Value" "C_Small"
+		(property "Value" "1nF"
 			(at 125.7363 92.71 90)
 			(effects
@@
 			)
 		)
-		(property "Value" "C_Small"
+		(property "Value" "1nF"
 			(at 125.7363 85.09 90)
 			(effects

Commit message: moon
Parts:
- C35: footprint Capacitor_SMD:C_0402_1005Metric -> Capacitor_SMD:C_0603_1608Metric
Changed lines of the file:
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@@
 			)
 		)
-		(property "Footprint" "Capacitor_SMD:C_0402_1005Metric"
+		(property "Footprint" "Capacitor_SMD:C_0603_1608Metric"
 			(at 148.59 67.31 0)
 			(effects
