File: LNA.kicad_sch (KiCad schematic)
At the start: 11 parts, among them Q2 BFP740F

Commit message: Rev 1 ready for review
Parts:
- C50: value 220 nF -> 140nF
- C51: value 43 pF -> 10pF
- C52: value 220 nF -> 220nF
- C53: value 3.3 pF -> 4.3 pF
- L16: value 200 nF -> 130nH
- L17: value 200 nF -> 260nH
- L18: value 200 nF -> 30nH
- R16: value 20k -> 100k
- R17: value 10 -> 50
- R18: value 50 -> ~; now not fitted; now left out of the parts list
Changed lines of the file:
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@@
 			)
 		)
-		(property "Value" "10"
+		(property "Value" "50"
 			(at 157.48 82.5499 0)
 			(effects
@@
 		(unit 1)
 		(exclude_from_sim no)
-		(in_bom yes)
-		(on_board yes)
-		(dnp no)
+		(in_bom no)
+		(on_board yes)
+		(dnp yes)
 		(fields_autoplaced yes)
 		(property "Reference" "R18"
@@
 			)
 		)
-		(property "Value" "50"
+		(property "Value" "~"
 			(at 177.8 102.8699 0)
 			(effects
@@
 			)
 		)
-		(property "Value" "200 nF"
+		(property "Value" "130nH"
 			(at 148.59 92.7099 0)
 			(effects
@@
 			)
 		)
-		(property "Value" "20k"
+		(property "Value" "100k"
 			(at 149.86 82.5499 0)
 			(effects
@@
 			)
 		)
-		(property "Value" "200 nF"
+		(property "Value" "30nH"
 			(at 156.21 114.2999 0)
 			(effects
@@
 			)
 		)
-		(property "Value" "220 nF"
+		(property "Value" "220nF"
 			(at 163.8363 82.55 90)
 			(effects
@@
 			)
 		)
-		(property "Value" "200 nF"
+		(property "Value" "260nH"
 			(at 156.21 92.7099 0)
 			(effects
@@
 			)
 		)
-		(property "Value" "220 nF"
+		(property "Value" "140nF"
 			(at 139.7063 82.55 90)
 			(effects
@@
 			)
 		)
-		(property "Value" "3.3 pF"
+		(property "Value" "4.3 pF"
 			(at 166.3763 93.98 90)
 			(effects
@@
 			)
 		)
-		(property "Value" "43 pF"
+		(property "Value" "10pF"
 			(at 139.7063 99.06 90)
 			(effects

Commit message: moon
Parts:
- L16: value 130nH -> 140nH
- L17: value 260nH -> 270nH
Changed lines of the file:
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@@
 			)
 		)
-		(property "Value" "130nH"
+		(property "Value" "140nH"
 			(at 148.59 92.7099 0)
 			(effects
@@
 			)
 		)
-		(property "Value" "260nH"
+		(property "Value" "270nH"
 			(at 156.21 92.7099 0)
 			(effects
