File: filter.kicad_sch (KiCad schematic)
At the start: 11 parts

Commit message: Rev 1 ready for review
Parts:
- C68, C72: value C -> 1.2pF
- C69, C71: value C -> 1nF
- C70: value C -> 0.36pF
- L20, L24: value L -> 1uH
- L21, L23: value L -> 1.2nH
- L22: value L -> 3.3uH
Changed lines of the file:
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@@
 			)
 		)
-		(property "Value" "L"
+		(property "Value" "3.3uH"
 			(at 130.81 92.71 90)
 			(effects
@@
 			)
 		)
-		(property "Value" "C"
+		(property "Value" "0.36pF"
 			(at 137.1663 91.44 90)
 			(effects
@@
 			)
 		)
-		(property "Value" "C"
+		(property "Value" "1.2pF"
 			(at 160.0263 91.44 90)
 			(effects
@@
 			)
 		)
-		(property "Value" "C"
+		(property "Value" "1nF"
 			(at 120.65 104.1462 0)
 			(effects
@@
 			)
 		)
-		(property "Value" "L"
+		(property "Value" "1.2nH"
 			(at 149.86 104.1399 0)
 			(effects
@@
 			)
 		)
-		(property "Value" "L"
+		(property "Value" "1.2nH"
 			(at 127 104.1399 0)
 			(effects
@@
 			)
 		)
-		(property "Value" "L"
+		(property "Value" "1uH"
 			(at 153.67 92.71 90)
 			(effects
@@
 			)
 		)
-		(property "Value" "L"
+		(property "Value" "1uH"
 			(at 107.95 92.71 90)
 			(effects
@@
 			)
 		)
-		(property "Value" "C"
+		(property "Value" "1nF"
 			(at 143.51 104.1462 0)
 			(effects
@@
 			)
 		)
-		(property "Value" "C"
+		(property "Value" "1.2pF"
 			(at 114.3063 91.44 90)
 			(effects

Commit message: load capacitor and shield paste
Parts:
- S3: footprint phase-detector:MS148-10 -> phase-detector:MS148-10F
Changed lines of the file:
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@@
 			)
 		)
-		(property "Footprint" "phase-detector:MS148-10"
+		(property "Footprint" "phase-detector:MS148-10F"
 			(at 119.634 126.492 0)
 			(effects
